File: classdamp/classdamp.kicad_sch (KiCad schematic)
At the start: 33 parts, among them J2 Conn_01x02_Pin

Commit message: Comparator stage
Parts:
- added C11, C12, C13, C14: 1n, Capacitor_THT:C_Disc_D5.0mm_W2.5mm_P5.00mm, symbol Device:C
- added R21, R22, R26, R27: 1k, Resistor_THT:R_Axial_DIN0207_L6.3mm_D2.5mm_P15.24mm_Horizontal, symbol Device:R
- added R23: 6.7k, Resistor_THT:R_Axial_DIN0207_L6.3mm_D2.5mm_P15.24mm_Horizontal, symbol Device:R
- added R24: 620, Resistor_THT:R_Axial_DIN0207_L6.3mm_D2.5mm_P15.24mm_Horizontal, symbol Device:R
- added R25: 10k, Resistor_THT:R_Axial_DIN0207_L6.3mm_D2.5mm_P15.24mm_Horizontal, symbol Device:R
- R14, R15, R16, R17, R18, R19, R20: footprint (none) -> Resistor_THT:R_Axial_DIN0207_L6.3mm_D2.5mm_P15.24mm_Horizontal
Connections:
- net +12V: now also C11.1, C13.1, R21.1, R22.1, R26.2, R27.1
- net GND: now also IC4.10 (Q4_E), IC4.13 (Q5_E_GND), C11.2, C13.2, C14.1, R24.1
- net at C10.1, R17.2, R18.1: now also IC4.2 (Q1_B)
- net at J2.1 (Pin_1), R20.1: now also C14.2
- net at IC4.1 (Q1_C): now also R22.2
- net at IC4.11 (Q4_C): now also R25.2, R26.1
- net at IC4.12 (Q5_B): now also R25.1
- net at IC4.14 (Q5_C): now also R27.2
- net at IC4.5 (Q2_C): now also C12.1, R21.2, R23.1, R24.2
- net at IC4.9 (Q4_B): now also C12.2, R23.2

Commit message: Test drawing in pcb and circuit fixes
Parts:
- removed R25: 10k, Resistor_THT:R_Axial_DIN0207_L6.3mm_D2.5mm_P15.24mm_Horizontal, symbol Device:R
- added C15: 1n, Capacitor_THT:C_Disc_D5.0mm_W2.5mm_P5.00mm, symbol Device:C
- added R28: 6.7k, Resistor_THT:R_Axial_DIN0207_L6.3mm_D2.5mm_P15.24mm_Horizontal, symbol Device:R
- added R29: 620, Resistor_THT:R_Axial_DIN0207_L6.3mm_D2.5mm_P15.24mm_Horizontal, symbol Device:R
- R13: value 1k -> 5k
- R9: value 33k -> 47k
Connections:
- net GND: now also R29.2
- net at IC4.12 (Q5_B): now also C15.1, R28.1
- net at IC4.1 (Q1_C), R22.2: now also C15.2, R28.2, R29.1

Commit message: PCB design done
Parts:
- added C16: 1000u, Capacitor_THT:CP_Radial_D8.0mm_P3.50mm, symbol Device:C_Small
- added C17, C18, C19, C20: 100n, Capacitor_THT:C_Disc_D5.0mm_W2.5mm_P5.00mm, symbol Device:C_Small
- added C21, C22, C25, C26: 1n, Capacitor_THT:C_Disc_D5.0mm_W2.5mm_P5.00mm, symbol Device:C
- added C23, C24, C27, C28: 100n, Capacitor_THT:C_Disc_D5.0mm_W2.5mm_P5.00mm, symbol Device:C
- added D1: 1N5822, Diode_THT:D_DO-35_SOD27_P7.62mm_Horizontal, symbol Diode:1N914
- added D2, D3, D4, D5, D6, D7: SS14, Diode_SMD:D_SMA_Handsoldering, symbol Diode:SS14
- added J1, J3: Conn_01x02_Pin, Connector:JWT_A3963_1x02_P3.96mm_Vertical, symbol Connector:Conn_01x02_Pin
- added L1: 100u, Inductor_THT:L_Toroid_Horizontal_D24.1mm_P23.10mm_Bourns_2200, symbol Device:L
- added L2, L3: 15u, Inductor_THT:L_Radial_D10.0mm_P5.00mm_Fastron_07M, symbol Device:L
- added Q1, Q12, Q14, Q6: S8550, Package_TO_SOT_THT:TO-92_Inline, symbol Transistor_BJT:Q_PNP_EBC
- added Q10, Q7, Q8, Q9: IPD135N03LGATMA1, Package_TO_SOT_SMD:TO-252-2, symbol Transistor_FET:Q_NMOS_GDS
- added Q11, Q13, Q4, Q5: S8050, Package_TO_SOT_THT:TO-92_Inline, symbol Transistor_BJT:Q_NPN_EBC
- added Q15, Q16, Q2, Q3: 2N5551, Package_TO_SOT_THT:TO-92_Inline, symbol Transistor_BJT:Q_NPN_EBC
- added R25, R30, R39, R40: 10k, Library:R_Axial_DIN0204_L3.6mm_D1.6mm_P2.54mm_Vertical, symbol Device:R
- added R31, R32, R37, R38: 1k, Library:R_Axial_DIN0204_L3.6mm_D1.6mm_P2.54mm_Vertical, symbol Device:R
- added R33, R36: 150, Library:R_Axial_DIN0204_L3.6mm_D1.6mm_P2.54mm_Vertical, symbol Device:R
- added R34, R35: 200, Library:R_Axial_DIN0204_L3.6mm_D1.6mm_P2.54mm_Vertical, symbol Device:R
- added R41, R42, R43, R44: 0, Resistor_THT:R_Axial_DIN0207_L6.3mm_D2.5mm_P15.24mm_Horizontal, symbol Device:R
- R14: value 1k -> 100
- R26, R27: value 1k -> 240
- R8: value 1k -> 330
- R9: value 47k -> 50k
Connections:
- net +12V: now also C27.2, C28.2, D1.1 (K), D2.2 (A), D5.2 (A), Q13.3 (C), Q4.3 (C), Q8.2 (D), Q9.2 (D), R31.2, R32.2, R37.2, R38.2, R43.1, R43.2, R44.1, R44.2
- net GND: now also C16.2, C17.2, C18.2, C19.2, C20.2, C27.1, C28.1, J3.1 (Pin_1), Q1.1 (E), Q10.3 (S), Q14.1 (E), Q15.1 (E), Q16.1 (E), Q2.1 (E), Q3.1 (E), Q7.3 (S)
- net at IC4.14 (Q5_C), R27.2: now also C21.2, C26.2, R25.2, R40.2, R41.1, R41.2
- net at IC4.11 (Q4_C), R26.1: now also C22.2, C25.2, R30.2, R39.2, R42.1, R42.2
- new net: J1.1 (Pin_1), L2.2
- new net: D3.1 (K), Q5.1 (E), Q6.3 (C), R34.2
- new net: Q3.3 (C), Q5.2 (B), Q6.2 (B), R32.1
- new net: J1.2 (Pin_2), L3.1
- new net: C16.1, C17.1, C18.1, C19.1, C20.1, D1.2 (A), L1.1
- new net: C21.1, Q3.2 (B), R25.1
- new net: C25.1, Q15.2 (B), R39.1
- new net: Q11.2 (B), Q12.2 (B), Q15.3 (C), R37.1
- new net: Q1.2 (B), Q2.3 (C), Q4.2 (B), R31.1
- new net: D6.1 (K), Q11.1 (E), Q12.3 (C), R35.2
- new net: Q13.2 (B), Q14.2 (B), Q16.3 (C), R38.1
- new net: D7.1 (K), Q13.1 (E), Q14.3 (C), R36.2
- new net: C22.1, Q2.2 (B), R30.1
- new net: D3.2 (A), Q8.1 (G), R34.1
- new net: D6.2 (A), Q9.1 (G), R35.1
- new net: D7.2 (A), Q10.1 (G), R36.1
- new net: D4.2 (A), Q7.1 (G), R33.1
- new net: D4.1 (K), Q1.3 (C), Q4.1 (E), R33.2
- new net: C26.1, Q16.2 (B), R40.1
- new net +12VA: J3.2 (Pin_2), L1.2
- new net PRI2_HI: C24.2, D5.1 (K), Q11.3 (C)
- new net PRI2_MID: C24.1, L2.1, Q10.2 (D), Q12.1 (E), Q9.3 (S)
- new net PRI_HI: C23.2, D2.1 (K), Q5.3 (C)
- new net PRI_MID: C23.1, L3.2, Q6.1 (E), Q7.2 (D), Q8.3 (S)
